File: Design_V1/MCU.kicad_sch (KiCad schematic)
At the start: 15 parts, among them J1 Conn_02x03_Counter_Clockwise, U1 RP2040, U2 W25Q128JVS

Commit message: Updated Project. Added testpoints, crystal and jumpers. Added Power block
Parts:
- removed J1: Conn_02x03_Counter_Clockwise, symbol Connector_Generic:Conn_02x03_Counter_Clockwise
- added C11, C12: 100nF, symbol Device:C_Small
- added C13: 1uF, symbol Device:C_Small
- added J1: Conn_02x04_Odd_Even, Connector_PinHeader_2.54mm:PinHeader_2x04_P2.54mm_Vertical_SMD, symbol Connector_Generic:Conn_02x04_Odd_Even
- added JP1: Jumper_2_Open, symbol Jumper:Jumper_2_Open
- added R3, R4: 1K, symbol Device:R_Small
- added R5: DNF, symbol Device:R_Small
- added TP1, TP10, TP2, TP3, TP4, TP5, TP6, TP7, TP8, TP9: TestPoint, symbol Connector:TestPoint
- added Y1: Crystal, symbol Device:Crystal
- C9: value 100nF -> 1uF
Connections:
- net +1V1: now also J1.6 (Pin_6)
- net +3V3: now also U1.44 (VREG_VIN), C13.1, J1.2 (Pin_2), R5.1
- net +5V: now also J1.4 (Pin_4)
- net GND: now also U1.57 (GND), C11.1, C12.1, C13.2, J1.8 (Pin_8), JP1.1 (A)
- net QSPI_CSN_U1_56: now also R4.2, R5.2, TP3.1
- net QSPI_SCLK_U1_52: now also TP4.1
- net QSPI_SD0_U1_53: now also TP5.1
- net QSPI_SD1_U1_55: now also TP6.1
- net QSPI_SD2_U1_54: now also TP7.1
- net QSPI_SD3_U1_51: now also TP8.1
- net RUN_U1_26: now also J1.1 (Pin_1)
- net SWCLK_U1_24: now also J1.3 (Pin_3)
- net SWD_U1_25: now also J1.5 (Pin_5)
- net USB_DM_U1_46: now also TP9.1
- net USB_DP_U1_47: now also TP10.1
- net XIN_U1_20: now also C11.2, TP1.1, Y1.2
- net XOUT_U1_21: now also R3.2, TP2.1
- net TESTEB_U1_19: now reaches U1.19 (TESTEN)
- net TESTEB_U1_19: now also J1.7 (Pin_7)
- new net: C12.2, R3.1, Y1.1
- new net: JP1.2 (B), R4.1
Other:
- moved on the sheet: C1, C10, C2, C3, C4, C5, C6, C7, C8, C9
