File: Design_V1/Design_V1.kicad_sch (KiCad schematic)
At the start: 0 parts

Commit message: Updated Ethernet
Other:
- sheet Ethernet ports: added ETH_MISO, ETH_MOSI, ETH_SCLK, ETH_SEN, ETH_nCS, ETH_nRD, ETH_nSCS, ETH_nWR; removed none
Changed lines of the file:
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@@
       (effects (font (size 1.27 1.27)) (justify left top))
+    )
+    (pin "ETH_SCLK" input (at 117.475 71.755 180)
+      (effects (font (size 1.27 1.27)) (justify left))
+    )
+    (pin "ETH_nSCS" input (at 117.475 74.295 180)
+      (effects (font (size 1.27 1.27)) (justify left))
+    )
+    (pin "ETH_SEN" input (at 117.475 76.835 180)
+      (effects (font (size 1.27 1.27)) (justify left))
+    )
+    (pin "ETH_nRD" input (at 117.475 79.375 180)
+      (effects (font (size 1.27 1.27)) (justify left))
+    )
+    (pin "ETH_MOSI" input (at 117.475 81.915 180)
+      (effects (font (size 1.27 1.27)) (justify left))
+    )
+    (pin "ETH_MISO" input (at 117.475 84.455 180)
+      (effects (font (size 1.27 1.27)) (justify left))
+    )
+    (pin "ETH_nCS" input (at 117.475 86.995 180)
+      (effects (font (size 1.27 1.27)) (justify left))
+    )
+    (pin "ETH_nWR" input (at 117.475 89.535 180)
+      (effects (font (size 1.27 1.27)) (justify left))
     )
   )
@@
       (reference "#PWR034") (unit 1) (value "+3.3VA") (footprint "")
     )
+    (path "/71070041-e598-4cf8-9b6e-932bbf134d95/777b310e-ae3f-48bb-bede-29564a6499c9"
+      (reference "#PWR035") (unit 1) (value "GND") (footprint "")
+    )
     (path "/9bd6305a-703c-44bf-adb0-bbf4076617c8/ed459d60-2755-4580-bbb0-62778a4d08b2"
       (reference "C1") (unit 1) (value "100nF") (footprint "")
@@
       (reference "C19") (unit 1) (value "10uF") (footprint "")
     )
+    (path "/71070041-e598-4cf8-9b6e-932bbf134d95/93b15f42-6572-4430-8476-baaaf8f8187d"
+      (reference "D1") (unit 1) (value "LED") (footprint "")
+    )
+    (path "/71070041-e598-4cf8-9b6e-932bbf134d95/da0ab733-fde3-4261-93bf-98604aae72f3"
+      (reference "D2") (unit 1) (value "LED") (footprint "")
+    )
+    (path "/71070041-e598-4cf8-9b6e-932bbf134d95/94a99495-a41b-4012-a49c-ae45fcdd20aa"
+      (reference "D3") (unit 1) (value "LED") (footprint "")
+    )
+    (path "/71070041-e598-4cf8-9b6e-932bbf134d95/41ddf282-f863-4a31-ac23-5171a3e7c7eb"
+      (reference "D4") (unit 1) (value "LED") (footprint "")
+    )
+    (path "/71070041-e598-4cf8-9b6e-932bbf134d95/939d3060-f00b-4c26-afbc-f90524736e5b"
+      (reference "D5") (unit 1) (value "LED") (footprint "")
+    )
+    (path "/71070041-e598-4cf8-9b6e-932bbf134d95/10020d56-9d89-48ea-a17b-a6dbb4f77037"
+      (reference "D6") (unit 1) (value "LED") (footprint "")
+    )
     (path "/9bd6305a-703c-44bf-adb0-bbf4076617c8/5b35bf9a-9013-4dc9-b3c3-371e481d9e79"
       (reference "J1") (unit 1) (value "Conn_02x04_Odd_Even") (footprint "Connector_PinHeader_2.54mm:PinHeader_2x04_P2.54mm_Vertical_SMD")
@@
       (reference "R5") (unit 1) (value "DNF") (footprint "")
     )
+    (path "/71070041-e598-4cf8-9b6e-932bbf134d95/42c18bd7-55e8-4975-ae73-4671ab75336e"
+      (reference "R6") (unit 1) (value "1K") (footprint "")
+    )
+    (path "/71070041-e598-4cf8-9b6e-932bbf134d95/6a7cec4f-d61c-4537-be1c-54adf0e627ad"
+      (reference "R7") (unit 1) (value "1K") (footprint "")
+    )
+    (path "/71070041-e598-4cf8-9b6e-932bbf134d95/4aac27a7-e070-46e4-bd09-900031612217"
+      (reference "R8") (unit 1) (value "1K") (footprint "")
+    )
+    (path "/71070041-e598-4cf8-9b6e-932bbf134d95/4961eff0-5cd2-426b-b9ef-0d427d00198e"
+      (reference "R9") (unit 1) (value "1K") (footprint "")
+    )
+    (path "/71070041-e598-4cf8-9b6e-932bbf134d95/9df7e6d2-3d47-4d46-94fd-ee52d9014f7c"
+      (reference "R10") (unit 1) (value "1K") (footprint "")
+    )
+    (path "/71070041-e598-4cf8-9b6e-932bbf134d95/7aabb704-ff64-45ed-92c2-6cf437cd0499"
+      (reference "R11") (unit 1) (value "1K") (footprint "")
+    )
     (path "/9bd6305a-703c-44bf-adb0-bbf4076617c8/4f7d8c71-9c89-47e1-bdd9-71ea2ff9470f"
