File: Design_V1/Ethernet.kicad_sch (KiCad schematic)
At the start: 9 parts, among them U3 W5100

Commit message: Updated Ethernet
Parts:
- added D1, D2, D3, D4, D5, D6: LED, symbol Device:LED
- added R10, R11, R6, R7, R8, R9: 1K, symbol Device:R_Small
Connections:
- net GND: now also D1.1 (K), D2.1 (K), D3.1 (K), D4.1 (K), D5.1 (K), D6.1 (K)
- net VCC1V8D_U1_15: now reaches U3.15 (VCC1V8D), U3.16 (VCC1V8D), U3.33 (VCC1V8D), U3.69 (VCC1V8D)
- net ETH_MISO: now reaches U3.27 (MISO)
- net ETH_MOSI: now reaches U3.28 (MOSI)
- net ETH_nSCS: now reaches U3.29 (~{SCS})
- net ETH_SCLK: now reaches U3.30 (SCLK)
- net ETH_SEN: now reaches U3.31 (SEN)
- net ETH_nCS: now reaches U3.55 (~{CS})
- net ETH_nINT: now reaches U3.56 (~{INT})
- net ETH_nWR: now reaches U3.57 (~{WR})
- net ETH_nRD: now reaches U3.58 (~{RD})
- net ETH_nRESET: now reaches U3.59 (~{RESET})
- net LINKLED: now reaches U3.66 (LINKLED)
- net LINKLED: now also R6.1
- net SPDLED: now reaches U3.67 (SPDLED)
- net SPDLED: now also R7.1
- net FDXLED: now reaches U3.70 (FDXLED)
- net FDXLED: now also R8.1
- net COLLED: now reaches U3.71 (COLLED)
- net COLLED: now also R9.1
- net RXLED: now reaches U3.72 (RXLED)
- net RXLED: now also R10.1
- net TXLED: now reaches U3.73 (TXLED)
- net TXLED: now also R11.1
- new net: D6.2 (A), R11.2
- new net: D4.2 (A), R9.2
- new net: D1.2 (A), R6.2
- new net: D3.2 (A), R8.2
- new net: D2.2 (A), R7.2
- new net: D5.2 (A), R10.2
